File: HB-OU-MP3-LED/HB-OU-MP3-LED_V1.2.brd (EAGLE design)
At the start: 76.2 x 100 mm, 19 parts, among them Q1 BC327, X1 MSTBA2, X2 MSTBA2

Commit message: Update HB-OU-MP3-LED_V1.2.brd
Parts:
- R1: value 1K -> 10K
Connections:
- net N$7: now also U$5.SWCLOSED; no longer U$5.SWOPEN
Routing:
- net N$7: track 16.8 -> 6.71 mm
Changed lines of the file:
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@@
 <attribute name="VALUE" x="22.225" y="24.13" size="1.27" layer="27" ratio="10"/>
 </element>
-<element name="R1" library="resistor" library_urn="urn:adsk.eagle:library:348" package="0309/10" package3d_urn="urn:adsk.eagle:package:23567/1" value="1K" x="29.21" y="27.94" smashed="yes">
+<element name="R1" library="resistor" library_urn="urn:adsk.eagle:library:348" package="0309/10" package3d_urn="urn:adsk.eagle:package:23567/1" value="10K" x="29.21" y="27.94" smashed="yes">
 <attribute name="NAME" x="25.019" y="29.845" size="1.27" layer="25" ratio="10"/>
 <attribute name="VALUE" x="26.035" y="27.2542" size="1.27" layer="27" ratio="10"/>
@@
 <signal name="N$7">
 <contactref element="U$4" pad="SPK2"/>
-<contactref element="U$5" pad="SWOPEN"/>
-<wire x1="29.47" y1="19.85" x2="31.75" y2="17.57" width="0.254" layer="16"/>
-<wire x1="31.75" y1="17.57" x2="31.75" y2="8.89" width="0.254" layer="16"/>
-<wire x1="31.75" y1="8.89" x2="34.29" y2="6.35" width="0.254" layer="16"/>
-<wire x1="34.29" y1="6.35" x2="35.56" y2="6.35" width="0.254" layer="16"/>
+<wire x1="35.56" y1="6.35" x2="34.29" y2="6.35" width="0.254" layer="16"/>
+<contactref element="U$5" pad="SWCLOSED"/>
+<wire x1="34.29" y1="6.35" x2="33.02" y2="6.35" width="0.1524" layer="16"/>
+<wire x1="31.52" y1="7.85" x2="29.47" y2="7.85" width="0.1524" layer="16"/>
+<wire x1="33.02" y1="6.35" x2="31.52" y2="7.85" width="0.1524" layer="16"/>
 </signal>
 <signal name="N$13">
