File: HB-OU-MP3-LED/HB-OU-MP3-LED_V1.2.sch (EAGLE design)
At the start: 19 parts, among them Q1 BC327, X1 MSTBA2, X2 MSTBA2

Commit message: Update HB-OU-MP3-LED_V1.2.sch
Parts:
- R1: value 1K -> 10K
Connections:
- net N$7: now also U$5.SWCLOSE; no longer U$5.SWOPEN
Changed lines of the file:
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@@
 <part name="X2" library="con-phoenix-508" library_urn="urn:adsk.eagle:library:176" deviceset="MSTBA2" device="" package3d_urn="urn:adsk.eagle:package:9615/1"/>
 <part name="Q1" library="transistor-pnp" library_urn="urn:adsk.eagle:library:399" deviceset="BC327" device="" package3d_urn="urn:adsk.eagle:package:29211/2"/>
-<part name="R1" library="resistor" library_urn="urn:adsk.eagle:library:348" deviceset="R-EU_" device="0309/10" package3d_urn="urn:adsk.eagle:package:23567/1" value="1K"/>
+<part name="R1" library="resistor" library_urn="urn:adsk.eagle:library:348" deviceset="R-EU_" device="0309/10" package3d_urn="urn:adsk.eagle:package:23567/1" value="10K"/>
 <part name="U$5" library="SRD-05VDC-SL-C" deviceset="RELAY" device="PTH"/>
 <part name="D1" library="diode" library_urn="urn:adsk.eagle:library:210" deviceset="1N4004" device="" package3d_urn="urn:adsk.eagle:package:43336/1"/>
@@
 <wire x1="213.36" y1="96.52" x2="213.36" y2="33.02" width="0.1524" layer="91"/>
 <wire x1="213.36" y1="33.02" x2="325.12" y2="33.02" width="0.1524" layer="91"/>
-<wire x1="325.12" y1="33.02" x2="325.12" y2="43.18" width="0.1524" layer="91"/>
-<pinref part="U$5" gate="G$1" pin="SWOPEN"/>
-<wire x1="325.12" y1="43.18" x2="322.58" y2="43.18" width="0.1524" layer="91"/>
-</segment>
-</net>
+<pinref part="U$5" gate="G$1" pin="SWCLOSE"/>
+<wire x1="322.58" y1="53.34" x2="325.12" y2="53.34" width="0.1524" layer="91"/>
+<wire x1="325.12" y1="53.34" x2="325.12" y2="33.02" width="0.1524" layer="91"/>
+</segment>
+</net>
