File: HB-OU-MP3-LED/HB-OU-MP3-LED_V1.3.brd (EAGLE design)
At the start: 76.2 x 100 mm, 23 parts, among them Q1 BC327, X1 MSTBA2, X2 MSTBA2

Commit message: Update HB-OU-MP3-LED_V1.3.brd
Parts:
- removed R1: 1K, resistor:0309/10
- removed X2: MSTBA2, con-phoenix-508:MSTBA2
- added X3: MSTBA3, con-phoenix-508:MSTBA3
- moved LED5 18.1 mm to (17.8, 61.0)
- moved CONFIG 13.1 mm to (12.7, 50.8)
- moved R5 12.6 mm to (24.1, 55.9), turned to 90 degrees
- moved JP1 10.2 mm to (5.08, 38.1)
- moved R2 4.02 mm to (38.1, 30.5)
- moved R3 4.02 mm to (38.1, 26.7)
- moved D1 1.27 mm to (16.5, 12.7)
- moved LED1 1.27 mm to (43.2, 6.35), turned to 270 degrees
- turned R4 to 270 degrees
- turned R6 to 270 degrees
Connections:
- net N$13: now also X3.2; no longer X2.2
- net N$20: now also U$5.SWOPEN, X3.3; no longer LED1.A, R6.1
- net N$5: now also R6.1; no longer R1.1, R6.2
- net N$6: now also X3.1; no longer X2.1
- net N$8: now also LED1.A, R6.2; no longer R1.2
Routing:
- net GND: track 0.00 -> 265.5 mm
- net RAW: track 0.00 -> 103.1 mm
- net VCC: track 0.00 -> 90.2 mm
- net N$5: track 0.00 -> 64.2 mm
- net GDO0: track 0.00 -> 52.2 mm
- net N$6: track 0.00 -> 48.9 mm
- net N$11: track 0.00 -> 34.7 mm
- net N$8: track 0.00 -> 34.7 mm
- net N$20: track 0.00 -> 34.0 mm
- net CSN: track 0.00 -> 31.1 mm
- net SCLK: track 0.00 -> 26.6 mm
- net N$1: track 0.00 -> 26.5 mm
- net SO: track 0.00 -> 25.6 mm
- net N$10: track 0.00 -> 23.8 mm
- net N$19: track 0.00 -> 20.3 mm
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Other:
- board text added: "CONFIG"
