File: HB-OU-MP3-LED/HB-OU-MP3-LED_V1.3.sch (EAGLE design)
At the start: 23 parts, among them Q1 BC327, X1 MSTBA2, X2 MSTBA2

Commit message: Update HB-OU-MP3-LED_V1.3.sch
Parts:
- removed R1: 1K, resistor:R-EU_0309/10
- removed X2: MSTBA2, con-phoenix-508:MSTBA2
- added X3: MSTBA3, con-phoenix-508:MSTBA3
Connections:
- net N$13: now also X3-2.1; no longer X2-2.1
- net N$20: now also U$5.SWOPEN, X3-3.1; no longer LED1.A, R6.1
- net N$5: now also R6.1; no longer R1.1, R6.2
- net N$6: now also X3-1.1; no longer X2-1.1
- net N$8: now also LED1.A, R6.2; no longer R1.2
Other:
- moved on the sheet: LED1, R6
