File: HB-Dis-EP-42BW/EAGLE/HB-Dis-EP-42BW.brd (EAGLE design)
At the start: 123 x 78.5 mm, 32 parts, among them Q1 16Mhz, X1 MSTBA2

Commit message: Update HB-Dis-EP-42BW.brd
Parts:
- added JP4: AVR-ISP-6VERT, avr-7:AVR-ISP-6
Connections:
- net GND: now also JP4.6; no longer J1.5
- net N$9: now also JP4.5
- net SCLK: now also JP4.3
- net SI: now also JP4.4
- net SO: now also JP4.1
- net VCC5.0: now also JP4.2
Routing:
- net VCC5.0: track 134.5 -> 189.3 mm, vias 1 -> 3
- net N$9: track 64.4 -> 98.8 mm
- net SCLK: track 27.0 -> 57.9 mm, vias 0 -> 1
- net SO: track 25.7 -> 51.4 mm, vias 0 -> 2
- net GND: track 471.0 -> 496.4 mm
- net SI: track 30.1 -> 34.3 mm
- net GDO0: track 28.5 -> 26.8 mm
- net CSN: track 21.2 -> 19.8 mm
