File: HB-Dis-EP-42BW/EAGLE/HB-Dis-EP-42BW.sch (EAGLE design)
At the start: 32 parts, among them Q1 16Mhz, X1 MSTBA2

Commit message: Update HB-Dis-EP-42BW.sch
Parts:
- added JP4: AVR-ISP-6VERT, avr-7:AVR-ISP-6VERT
Connections:
- net GND: now also JP4.6; no longer J1.CTS
- net N$9: now also JP4.5
- net SCLK: now also JP4.3
- net SI: now also JP4.4
- net SO: now also JP4.1
- net VCC5.0: now also JP4.2
Changed lines of the file:
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@@
 <part name="C4" library="resistor" library_urn="urn:adsk.eagle:library:348" deviceset="C-EU" device="025-024X044" package3d_urn="urn:adsk.eagle:package:23630/1" value="0,1yF"/>
 <part name="C5" library="resistor" library_urn="urn:adsk.eagle:library:348" deviceset="C-EU" device="025-024X044" package3d_urn="urn:adsk.eagle:package:23630/1" value="0,1yF"/>
+<part name="JP4" library="avr-7" deviceset="AVR-ISP-6" device="VERT"/>
 </parts>
 <sheets>
@@
 <attribute name="NAME" x="-1.524" y="68.199" size="1.778" layer="95" rot="R180"/>
 <attribute name="VALUE" x="-1.524" y="73.279" size="1.778" layer="96" rot="R180"/>
+</instance>
+<instance part="JP4" gate="G$1" x="35.56" y="-27.94" smashed="yes">
+<attribute name="NAME" x="29.21" y="-21.59" size="1.778" layer="95" ratio="10"/>
 </instance>
 </instances>
@@
 <label x="81.28" y="-33.02" size="1.778" layer="95" rot="R270"/>
 <pinref part="IC1" gate="G$1" pin="MOSI/ICP3/PCINT13"/>
-<wire x1="81.28" y1="-48.26" x2="81.28" y2="58.42" width="0.1524" layer="91"/>
+<wire x1="81.28" y1="-48.26" x2="81.28" y2="-27.94" width="0.1524" layer="91"/>
+<wire x1="81.28" y1="-27.94" x2="81.28" y2="58.42" width="0.1524" layer="91"/>
 <wire x1="81.28" y1="58.42" x2="55.88" y2="58.42" width="0.1524" layer="91"/>
+<pinref part="JP4" gate="G$1" pin="4"/>
+<wire x1="40.64" y1="-27.94" x2="81.28" y2="-27.94" width="0.1524" layer="91"/>
+<junction x="81.28" y="-27.94"/>
 </segment>
 </net>
@@
 <pinref part="IC1" gate="G$1" pin="MISO/OC3A/PCINT14"/>
 <wire x1="55.88" y1="55.88" x2="76.2" y2="55.88" width="0.1524" layer="91"/>
-<wire x1="76.2" y1="55.88" x2="76.2" y2="-48.26" width="0.1524" layer="91"/>
+<wire x1="76.2" y1="55.88" x2="76.2" y2="-17.78" width="0.1524" layer="91"/>
+<pinref part="JP4" gate="G$1" pin="1"/>
+<wire x1="76.2" y1="-17.78" x2="76.2" y2="-48.26" width="0.1524" layer="91"/>
+<wire x1="30.48" y1="-25.4" x2="22.86" y2="-25.4" width="0.1524" layer="91"/>
+<wire x1="22.86" y1="-25.4" x2="22.86" y2="-17.78" width="0.1524" layer="91"/>
+<wire x1="22.86" y1="-17.78" x2="76.2" y2="-17.78" width="0.1524" layer="91"/>
+<junction x="76.2" y="-17.78"/>
 </segment>
 </net>
@@
 <pinref part="IC1" gate="G$1" pin="SCK/OC3B/PCINT15"/>
 <wire x1="55.88" y1="53.34" x2="78.74" y2="53.34" width="0.1524" layer="91"/>
-<wire x1="78.74" y1="53.34" x2="78.74" y2="-48.26" width="0.1524" layer="91"/>
+<wire x1="78.74" y1="53.34" x2="78.74" y2="-15.24" width="0.1524" layer="91"/>
+<pinref part="JP4" gate="G$1" pin="3"/>
+<wire x1="78.74" y1="-15.24" x2="78.74" y2="-48.26" width="0.1524" layer="91"/>
+<wire x1="30.48" y1="-27.94" x2="20.32" y2="-27.94" width="0.1524" layer="91"/>
+<wire x1="20.32" y1="-27.94" x2="20.32" y2="-15.24" width="0.1524" layer="91"/>
+<wire x1="20.32" y1="-15.24" x2="78.74" y2="-15.24" width="0.1524" layer="91"/>
+<junction x="78.74" y="-15.24"/>
 </segment>
 </net>
@@
 <wire x1="-20.32" y1="-40.64" x2="-20.32" y2="-38.1" width="0.1524" layer="91"/>
 <junction x="-20.32" y="7.62"/>
-<pinref part="J1" gate="G$1" pin="CTS"/>
 <wire x1="-20.32" y1="-38.1" x2="-20.32" y2="7.62" width="0.1524" layer="91"/>
-<wire x1="-2.54" y1="-40.64" x2="-2.54" y2="-38.1" width="0.1524" layer="91"/>
-<wire x1="-2.54" y1="-38.1" x2="-20.32" y2="-38.1" width="0.1524" layer="91"/>
 <junction x="-20.32" y="-38.1"/>
 <pinref part="C4" gate="G$1" pin="1"/>
@@
 <junction x="149.86" y="43.18"/>
 <pinref part="U$1" gate="G$1" pin="2"/>
+<pinref part="JP4" gate="G$1" pin="6"/>
+<wire x1="40.64" y1="-30.48" x2="45.72" y2="-30.48" width="0.1524" layer="91"/>
+<wire x1="45.72" y1="-30.48" x2="45.72" y2="-38.1" width="0.1524" layer="91"/>
+<wire x1="45.72" y1="-38.1" x2="-20.32" y2="-38.1" width="0.1524" layer="91"/>
 </segment>
 </net>
@@
 <wire x1="0" y1="76.2" x2="0" y2="73.66" width="0.1524" layer="91"/>
 <junction x="0" y="76.2"/>
+<pinref part="JP4" gate="G$1" pin="5"/>
+<wire x1="30.48" y1="-30.48" x2="15.24" y2="-30.48" width="0.1524" layer="91"/>
+<wire x1="15.24" y1="-30.48" x2="15.24" y2="-10.16" width="0.1524" layer="91"/>
+<wire x1="15.24" y1="-10.16" x2="-5.08" y2="-10.16" width="0.1524" layer="91"/>
+<wire x1="-5.08" y1="-10.16" x2="-5.08" y2="76.2" width="0.1524" layer="91"/>
+<wire x1="-5.08" y1="76.2" x2="0" y2="76.2" width="0.1524" layer="91"/>
 </segment>
 </net>
@@
 <label x="86.36" y="109.22" size="1.778" layer="95"/>
 <pinref part="J1" gate="G$1" pin="VCC"/>
-<wire x1="0" y1="-40.64" x2="0" y2="-27.94" width="0.1524" layer="91"/>
+<wire x1="0" y1="-40.64" x2="0" y2="-35.56" width="0.1524" layer="91"/>
+<wire x1="0" y1="-35.56" x2="0" y2="-27.94" width="0.1524" layer="91"/>
 <wire x1="0" y1="-27.94" x2="-25.4" y2="-27.94" width="0.1524" layer="91"/>
 <wire x1="-25.4" y1="-27.94" x2="-25.4" y2="114.3" width="0.1524" layer="91"/>
@@
 <wire x1="177.8" y1="30.48" x2="198.12" y2="30.48" width="0.1524" layer="91"/>
 <label x="185.42" y="30.48" size="1.778" layer="95"/>
-</segment>
-</net>
+<pinref part="JP4" gate="G$1" pin="2"/>
+<wire x1="40.64" y1="-25.4" x2="53.34" y2="-25.4" width="0.1524" layer="91"/>
+<wire x1="53.34" y1="-25.4" x2="53.34" y2="-35.56" width="0.1524" layer="91"/>
+<wire x1="53.34" y1="-35.56" x2="0" y2="-35.56" width="0.1524" layer="91"/>
+<junction x="0" y="-35.56"/>
+</segment>
+</net>
