File: HM-ES-PMSw1-Pl_GosundSP1/EAGLE/HB-power_v1.3.brd (EAGLE design)
At the start: 71.1 x 100 mm, 39 parts, among them IC1 ATMEGA644-10PU, IC4 HLW8012, Q1 16Mhz, T1 BC547, X1 MSTBA2, X2 MSTBA3

Commit message: Update HB-power_v1.3.brd
Parts:
- added JP2: AVR-ISP-6VERT, avr-7:AVR-ISP-6
Connections:
- net GND: now also JP2.6
- net N$26: now also JP2.2
- net N$27: now also JP2.5
- net SCLK: now also JP2.3
- net SI: now also JP2.4
- net SO: now also JP2.1
Routing:
- net SI: track 25.9 -> 67.3 mm
- net SCLK: track 31.8 -> 66.0 mm
- net SO: track 28.7 -> 58.2 mm
- net N$26: track 141.4 -> 169.4 mm
- net N$27: track 62.0 -> 88.7 mm, vias 0 -> 1
- net GND: track 269.3 -> 293.3 mm, vias 2 -> 3
Changed lines of the file:
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@@
 <hole x="3.81" y="3.81" drill="3.5"/>
 <hole x="67.31" y="3.81" drill="3.5"/>
-<text x="62.23" y="57.15" size="2.54" layer="25" rot="R90">HM-ES-PMSw1-PI</text>
-<text x="67.945" y="73.66" size="2.54" layer="25" rot="R90">V1.3</text>
+<text x="61.595" y="54.61" size="2.54" layer="25" rot="R90">HM-ES-PMSw1-PI</text>
+<text x="68.58" y="69.85" size="2.54" layer="25" rot="R90">V1.3</text>
 </plain>
 <attributes>
@@
 <attribute name="VALUE" x="26.035" y="95.9358" size="1.27" layer="27" ratio="10" rot="R180"/>
 </element>
+<element name="JP2" library="avr-7" package="AVR-ISP-6" value="AVR-ISP-6VERT" x="63.5" y="90.17" smashed="yes">
+<attribute name="NAME" x="59.69" y="85.725" size="1.27" layer="25" ratio="10"/>
+<attribute name="VALUE" x="57.15" y="92.71" size="1.27" layer="27" ratio="12"/>
+</element>
 </elements>
 <signals>
@@
 <wire x1="35.56" y1="83.185" x2="37.465" y2="81.28" width="0.254" layer="16"/>
 <wire x1="37.465" y1="81.28" x2="39.37" y2="81.28" width="0.254" layer="16"/>
+<contactref element="JP2" pad="4"/>
+<wire x1="63.5" y1="91.44" x2="63.5" y2="94.615" width="0.1524" layer="1"/>
+<wire x1="60.325" y1="97.79" x2="48.895" y2="97.79" width="0.1524" layer="1"/>
+<wire x1="48.895" y1="97.79" x2="43.815" y2="92.71" width="0.1524" layer="1"/>
+<wire x1="43.815" y1="92.71" x2="43.815" y2="82.55" width="0.1524" layer="1"/>
+<wire x1="43.815" y1="82.55" x2="42.545" y2="81.28" width="0.1524" layer="1"/>
+<wire x1="42.545" y1="81.28" x2="39.37" y2="81.28" width="0.1524" layer="1"/>
+<wire x1="63.5" y1="94.615" x2="60.325" y2="97.79" width="0.1524" layer="1"/>
 </signal>
 <signal name="SO">
@@
 <wire x1="34.925" y1="78.74" x2="39.37" y2="78.74" width="0.254" layer="16"/>
 <wire x1="12.97" y1="80.01" x2="33.655" y2="80.01" width="0.254" layer="16"/>
+<contactref element="JP2" pad="1"/>
+<wire x1="60.96" y1="88.9" x2="60.96" y2="82.55" width="0.1524" layer="16"/>
+<wire x1="44.45" y1="80.01" x2="43.18" y2="78.74" width="0.1524" layer="16"/>
+<wire x1="43.18" y1="78.74" x2="39.37" y2="78.74" width="0.1524" layer="16"/>
+<wire x1="60.96" y1="82.55" x2="58.42" y2="80.01" width="0.1524" layer="16"/>
+<wire x1="58.42" y1="80.01" x2="44.45" y2="80.01" width="0.1524" layer="16"/>
 </signal>
 <signal name="SCLK">
@@
 <wire x1="36.83" y1="76.2" x2="39.37" y2="76.2" width="0.254" layer="1"/>
 <wire x1="33.02" y1="83.185" x2="35.56" y2="80.645" width="0.254" layer="1"/>
+<contactref element="JP2" pad="3"/>
+<wire x1="63.5" y1="88.9" x2="63.5" y2="80.645" width="0.1524" layer="16"/>
+<wire x1="45.085" y1="77.47" x2="43.815" y2="76.2" width="0.1524" layer="16"/>
+<wire x1="43.815" y1="76.2" x2="39.37" y2="76.2" width="0.1524" layer="16"/>
+<wire x1="63.5" y1="80.645" x2="60.325" y2="77.47" width="0.1524" layer="16"/>
+<wire x1="60.325" y1="77.47" x2="45.085" y2="77.47" width="0.1524" layer="16"/>
 </signal>
 <signal name="L">
@@
 <wire x1="43.815" y1="31.115" x2="43.815" y2="29.845" width="0.254" layer="1"/>
 <wire x1="43.815" y1="29.845" x2="41.95" y2="27.98" width="0.254" layer="1"/>
-<wire x1="41.95" y1="27.98" x2="41.91" y2="27.94" width="0.254" layer="1"/>
 <via x="41.95" y="27.98" extent="1-16" drill="0.35"/>
+<contactref element="JP2" pad="2"/>
+<wire x1="60.96" y1="91.44" x2="59.055" y2="91.44" width="0.1524" layer="1"/>
+<wire x1="59.055" y1="91.44" x2="57.785" y2="90.17" width="0.1524" layer="1"/>
+<wire x1="57.785" y1="69.215" x2="57.15" y2="68.58" width="0.1524" layer="1"/>
+<wire x1="57.15" y1="68.58" x2="54.61" y2="68.58" width="0.1524" layer="1"/>
+<wire x1="57.785" y1="90.17" x2="57.785" y2="69.215" width="0.1524" layer="1"/>
 </signal>
 <signal name="N$27">
@@
 <wire x1="56.515" y1="67.31" x2="50.165" y2="67.31" width="0.254" layer="16"/>
 <wire x1="39.37" y1="39.37" x2="41.91" y2="39.37" width="0.254" layer="16"/>
+<contactref element="JP2" pad="5"/>
+<wire x1="66.04" y1="88.9" x2="66.04" y2="74.93" width="0.1524" layer="1"/>
+<wire x1="58.42" y1="67.31" x2="56.515" y2="67.31" width="0.1524" layer="1"/>
+<via x="56.515" y="67.31" extent="1-16" drill="0.35"/>
+<wire x1="66.04" y1="74.93" x2="58.42" y2="67.31" width="0.1524" layer="1"/>
 </signal>
 <signal name="N$24">
@@
 <wire x1="17.78" y1="81.2" x2="17.78" y2="77.47" width="0.254" layer="1"/>
 <wire x1="29.21" y1="31.75" x2="29.21" y2="33.655" width="0.1524" layer="1"/>
+<contactref element="JP2" pad="6"/>
+<wire x1="66.04" y1="91.44" x2="67.31" y2="91.44" width="0.1524" layer="1"/>
+<wire x1="67.31" y1="91.44" x2="68.58" y2="90.17" width="0.1524" layer="1"/>
+<wire x1="68.58" y1="90.17" x2="68.58" y2="75.565" width="0.1524" layer="1"/>
+<wire x1="68.58" y1="75.565" x2="64.135" y2="71.12" width="0.1524" layer="1"/>
+<via x="64.135" y="71.12" extent="1-16" drill="0.35"/>
 </signal>
 <signal name="N$34">
