File: HB-UNI-SenAct-4-4-RC/EAGLE/HB-UNI-SenAct-4-4-RC_V3.0.brd (EAGLE design)
At the start: 86.3 x 100 mm, 36 parts, among them IC1 ULN2803, X1 MSTBA2, X2 MSTBA3, X3 MSTBA3, X4 MSTBA3, X5 MSTBA3, X6 MSTBA2, X7 MSTBA2, X8 MSTBA2, X9 MSTBA2

Commit message: Update HB-UNI-SenAct-4-4-RC_V3.0.brd
Parts:
- F1: value (none) -> F2
- F2: value (none) -> F1
Changed lines of the file:
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@@
 <attribute name="VALUE" x="44.323" y="35.4965" size="1.27" layer="27" ratio="10" rot="R90"/>
 </element>
-<element name="F1" library="fuse" library_urn="urn:adsk.eagle:library:233" package="SH22,5A" package3d_urn="urn:adsk.eagle:package:14070/1" value="" x="65.9765" y="86.4235" smashed="yes" rot="R90">
+<element name="F1" library="fuse" library_urn="urn:adsk.eagle:library:233" package="SH22,5A" package3d_urn="urn:adsk.eagle:package:14070/1" value="F2" x="65.9765" y="86.4235" smashed="yes" rot="R90">
 <attribute name="MF" value="" x="133.2865" y="111.8235" size="1.778" layer="27" rot="R90" display="off"/>
 <attribute name="MPN" value="0031.7701.11" x="133.2865" y="111.8235" size="1.778" layer="27" rot="R90" display="off"/>
 <attribute name="OC_FARNELL" value="unknown" x="133.2865" y="111.8235" size="1.778" layer="27" rot="R90" display="off"/>
 <attribute name="OC_NEWARK" value="04F1224" x="133.2865" y="111.8235" size="1.778" layer="27" rot="R90" display="off"/>
-<attribute name="VALUE" x="73.5965" y="86.4489" size="1.778" layer="27" ratio="10" rot="R90"/>
+<attribute name="VALUE" x="73.5965" y="93.4339" size="1.778" layer="27" ratio="10" rot="R90"/>
 </element>
-<element name="F2" library="fuse" library_urn="urn:adsk.eagle:library:233" package="SH22,5A" package3d_urn="urn:adsk.eagle:package:14070/1" value="" x="14.0335" y="86.4235" smashed="yes" rot="R90">
+<element name="F2" library="fuse" library_urn="urn:adsk.eagle:library:233" package="SH22,5A" package3d_urn="urn:adsk.eagle:package:14070/1" value="F1" x="14.0335" y="86.4235" smashed="yes" rot="R90">
 <attribute name="MF" value="" x="81.3435" y="138.4935" size="1.778" layer="27" rot="R90" display="off"/>
 <attribute name="MPN" value="0031.7701.11" x="81.3435" y="138.4935" size="1.778" layer="27" rot="R90" display="off"/>
 <attribute name="OC_FARNELL" value="unknown" x="81.3435" y="138.4935" size="1.778" layer="27" rot="R90" display="off"/>
 <attribute name="OC_NEWARK" value="04F1224" x="81.3435" y="138.4935" size="1.778" layer="27" rot="R90" display="off"/>
-<attribute name="VALUE" x="21.6535" y="86.4489" size="1.778" layer="27" ratio="10" rot="R90"/>
+<attribute name="VALUE" x="7.6835" y="91.8464" size="1.778" layer="27" ratio="10" rot="R90"/>
 </element>
 <element name="LED1" library="led" library_urn="urn:adsk.eagle:library:259" package="LED3MM" package3d_urn="urn:adsk.eagle:package:15797/1" value="" x="54.991" y="68.326" smashed="yes" rot="R90">

Commit message: Update HB-UNI-SenAct-4-4-RC_V3.0.brd
Parts:
- RL2: value RELAYPTH -> RL2
- renumbered U$4 to RL1, U$5 to RL2, U$6 to RL3, U$7 to RL4
Changed lines of the file:
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@@
 <attribute name="VALUE" x="1.524" y="89.535" size="1.27" layer="27" ratio="10" rot="R270"/>
 </element>
-<element name="U$4" library="SRD-05VDC-SL-C" package="SRD-05VDC-SL-C" value="RELAYPTH" x="67.1195" y="65.5955" smashed="yes"/>
-<element name="U$5" library="SRD-05VDC-SL-C" package="SRD-05VDC-SL-C" value="RELAYPTH" x="67.183" y="49.4665" smashed="yes"/>
-<element name="U$6" library="SRD-05VDC-SL-C" package="SRD-05VDC-SL-C" value="RELAYPTH" x="67.183" y="33.0835" smashed="yes"/>
-<element name="U$7" library="SRD-05VDC-SL-C" package="SRD-05VDC-SL-C" value="RELAYPTH" x="67.183" y="15.8115" smashed="yes"/>
+<element name="RL1" library="SRD-05VDC-SL-C" package="SRD-05VDC-SL-C" value="RELAYPTH" x="67.1195" y="65.5955" smashed="yes">
+<attribute name="NAME" x="67.1195" y="69.4055" size="1.6764" layer="25"/>
+</element>
+<element name="RL2" library="SRD-05VDC-SL-C" package="SRD-05VDC-SL-C" value="RL2" x="67.183" y="49.4665" smashed="yes">
+<attribute name="NAME" x="67.183" y="52.959" size="1.6764" layer="25"/>
+</element>
+<element name="RL3" library="SRD-05VDC-SL-C" package="SRD-05VDC-SL-C" value="RELAYPTH" x="67.183" y="33.0835" smashed="yes">
+<attribute name="NAME" x="67.183" y="35.6235" size="1.6764" layer="25"/>
+</element>
+<element name="RL4" library="SRD-05VDC-SL-C" package="SRD-05VDC-SL-C" value="RELAYPTH" x="67.183" y="15.8115" smashed="yes">
+<attribute name="NAME" x="67.183" y="18.034" size="1.6764" layer="25"/>
+</element>
 <element name="X2" library="con-phoenix-508" library_urn="urn:adsk.eagle:library:176" package="MSTBA3" package3d_urn="urn:adsk.eagle:package:9608/1" value="MSTBA3" x="84.3915" y="67.6275" smashed="yes" rot="R90">
 <attribute name="MF" value="FARNELL" x="84.3915" y="67.6275" size="1.778" layer="27" rot="R90" display="off"/>
@@
 <contactref element="IC1" pad="10"/>
 <contactref element="F2" pad="2"/>
-<contactref element="U$7" pad="COIL0"/>
-<contactref element="U$6" pad="COIL0"/>
-<contactref element="U$4" pad="COIL0"/>
-<contactref element="U$5" pad="COIL0"/>
+<contactref element="RL4" pad="COIL0"/>
+<contactref element="RL3" pad="COIL0"/>
+<contactref element="RL1" pad="COIL0"/>
+<contactref element="RL2" pad="COIL0"/>
 <contactref element="R1" pad="2"/>
 <contactref element="R2" pad="2"/>
@@
 <signal name="N$22">
 <contactref element="X5" pad="2"/>
-<contactref element="U$7" pad="SWCOMMON"/>
+<contactref element="RL4" pad="SWCOMMON"/>
 <wire x1="59.793" y1="15.6915" x2="79.368" y2="15.6915" width="2.54" layer="1"/>
 <wire x1="79.368" y1="15.6915" x2="79.4385" y2="15.621" width="2.54" layer="1"/>
@@
 <signal name="N$26">
 <contactref element="X4" pad="2"/>
-<contactref element="U$6" pad="SWCOMMON"/>
+<contactref element="RL3" pad="SWCOMMON"/>
 <wire x1="59.793" y1="32.9635" x2="79.382" y2="32.9635" width="2.54" layer="1"/>
 <wire x1="79.382" y1="32.9635" x2="79.4385" y2="33.02" width="2.54" layer="1"/>
 </signal>
 <signal name="N$29">
-<contactref element="U$5" pad="SWCOMMON"/>
+<contactref element="RL2" pad="SWCOMMON"/>
 <contactref element="X3" pad="2"/>
 <wire x1="59.793" y1="49.3465" x2="65.539" y2="49.3465" width="2.54" layer="1"/>
@@
 </signal>
 <signal name="N$32">
-<contactref element="U$4" pad="SWCOMMON"/>
+<contactref element="RL1" pad="SWCOMMON"/>
 <contactref element="X2" pad="2"/>
 <wire x1="59.7295" y1="65.4755" x2="61.2465" y2="66.9925" width="2.54" layer="1"/>
@@
 <signal name="N$34">
 <contactref element="IC1" pad="18"/>
-<contactref element="U$4" pad="COIL1"/>
+<contactref element="RL1" pad="COIL1"/>
 <contactref element="LED1" pad="K"/>
 <wire x1="56.675" y1="71.1835" x2="56.5785" y2="71.1835" width="0.254" layer="16"/>
@@
 </signal>
 <signal name="N$35">
-<contactref element="U$5" pad="COIL1"/>
+<contactref element="RL2" pad="COIL1"/>
 <contactref element="IC1" pad="17"/>
 <contactref element="LED2" pad="K"/>
@@
 <signal name="N$36">
 <contactref element="IC1" pad="16"/>
-<contactref element="U$6" pad="COIL1"/>
+<contactref element="RL3" pad="COIL1"/>
 <contactref element="LED3" pad="K"/>
 <wire x1="49.9745" y1="52.6415" x2="51.181" y2="52.6415" width="0.254" layer="16"/>
@@
 <signal name="N$37">
 <contactref element="IC1" pad="15"/>
-<contactref element="U$7" pad="COIL1"/>
+<contactref element="RL4" pad="COIL1"/>
 <contactref element="LED4" pad="K"/>
 <wire x1="55.245" y1="17.4625" x2="57.564" y2="17.4625" width="0.254" layer="16"/>
@@
 </signal>
 <signal name="N$21">
-<contactref element="U$6" pad="SWCLOSED"/>
+<contactref element="RL3" pad="SWCLOSED"/>
 <contactref element="X4" pad="1"/>
 <wire x1="73.793" y1="26.9635" x2="74.7695" y2="27.94" width="2.54" layer="1"/>
@@
 </signal>
 <signal name="N$23">
-<contactref element="U$6" pad="SWOPEN"/>
+<contactref element="RL3" pad="SWOPEN"/>
 <contactref element="X4" pad="3"/>
 <wire x1="73.793" y1="38.9635" x2="74.6565" y2="38.1" width="2.54" layer="1"/>
@@
 <signal name="N$25">
 <contactref element="X5" pad="1"/>
-<contactref element="U$7" pad="SWCLOSED"/>
+<contactref element="RL4" pad="SWCLOSED"/>
 <wire x1="73.793" y1="9.6915" x2="74.6425" y2="10.541" width="2.54" layer="1"/>
 <wire x1="74.6425" y1="10.541" x2="79.4385" y2="10.541" width="2.54" layer="1"/>
 </signal>
 <signal name="N$27">
-<contactref element="U$7" pad="SWOPEN"/>
+<contactref element="RL4" pad="SWOPEN"/>
 <contactref element="X5" pad="3"/>
 <wire x1="73.793" y1="21.6915" x2="74.7835" y2="20.701" width="2.54" layer="1"/>
@@
 </signal>
 <signal name="N$28">
-<contactref element="U$5" pad="SWOPEN"/>
+<contactref element="RL2" pad="SWOPEN"/>
 <contactref element="X3" pad="3"/>
 <wire x1="73.793" y1="55.3465" x2="79.286" y2="55.3465" width="2.54" layer="1"/>
@@
 <signal name="N$30">
 <contactref element="X3" pad="1"/>
-<contactref element="U$5" pad="SWCLOSED"/>
+<contactref element="RL2" pad="SWCLOSED"/>
 <wire x1="73.793" y1="43.3465" x2="75.722" y2="45.2755" width="2.54" layer="1"/>
 <wire x1="75.722" y1="45.2755" x2="79.375" y2="45.2755" width="2.54" layer="1"/>
 </signal>
 <signal name="N$31">
-<contactref element="U$4" pad="SWOPEN"/>
+<contactref element="RL1" pad="SWOPEN"/>
 <contactref element="X2" pad="3"/>
 <wire x1="73.7295" y1="71.4755" x2="74.9615" y2="72.7075" width="2.54" layer="1"/>
@@
 <signal name="N$33">
 <contactref element="X2" pad="1"/>
-<contactref element="U$4" pad="SWCLOSED"/>
+<contactref element="RL1" pad="SWCLOSED"/>
 <wire x1="73.7295" y1="59.4755" x2="76.8015" y2="62.5475" width="2.54" layer="1"/>
 <wire x1="76.8015" y1="62.5475" x2="79.3115" y2="62.5475" width="2.54" layer="1"/>
