File: HB-OU-MP3-LED/EAGLE/HB-OU-MP3-LED_V1.3.sch (EAGLE design)
At the start: 22 parts, among them Q1 BC327, X1 MSTBA2, X3 MSTBA3

Commit message: Update HB-OU-MP3-LED_V1.3.sch
Parts:
- added R1: 10K, resistor:R-EU_0309/10
Connections:
- new net N$21: LED1.C, OK1.A
- new net N$22: Q1.B, R4.2
- net GND: now also R1.1; no longer LED1.C, OK1.EMIT
- net N$13: now also U$5.SWCLOSE; no longer U$5.SWCOMMON
- net N$16: now also OK1.EMIT, R1.2, R4.1; no longer OK1.COL, Q1.B, R4.2
- net N$7: now also U$5.SWCOMMON; no longer U$5.SWCLOSE
- net N$8: no longer OK1.A
- net RAW: now also OK1.COL; no longer R4.1
Other:
- moved on the sheet: D1, LED1, Q1, R4, U$5

Commit message: Update HB-OU-MP3-LED_V1.3.sch
Parts:
- D1: value 1N4004 -> 1N4007
- renumbered JP1 to RGB, LED5 to LED2, U$5 to RL1
Changed lines of the file:
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@@
 <part name="CONFIG" library="SparkFun-Switches" library_urn="urn:adsk.eagle:library:535" deviceset="MOMENTARY-SWITCH-SPST" device="-PTH-6.0MM-KIT" package3d_urn="urn:adsk.eagle:package:40170/1"/>
 <part name="R5" library="resistor" library_urn="urn:adsk.eagle:library:348" deviceset="R-EU_" device="0309/10" package3d_urn="urn:adsk.eagle:package:23567/1" value="470"/>
-<part name="LED5" library="led" library_urn="urn:adsk.eagle:library:259" deviceset="LED" device="3MM" package3d_urn="urn:adsk.eagle:package:15797/1"/>
+<part name="LED2" library="led" library_urn="urn:adsk.eagle:library:259" deviceset="LED" device="3MM" package3d_urn="urn:adsk.eagle:package:15797/1"/>
 <part name="X1" library="con-phoenix-508" library_urn="urn:adsk.eagle:library:176" deviceset="MSTBA2" device="" package3d_urn="urn:adsk.eagle:package:9615/1"/>
 <part name="U$4" library="DFPlayer_v1" deviceset="DFPLAYER" device=""/>
-<part name="JP1" library="jumper" library_urn="urn:adsk.eagle:library:252" deviceset="JP2E" device="" package3d_urn="urn:adsk.eagle:package:15452/1"/>
+<part name="RGB" library="jumper" library_urn="urn:adsk.eagle:library:252" deviceset="JP2E" device="" package3d_urn="urn:adsk.eagle:package:15452/1"/>
 <part name="Q1" library="transistor-pnp" library_urn="urn:adsk.eagle:library:399" deviceset="BC327" device="" package3d_urn="urn:adsk.eagle:package:29211/2"/>
-<part name="U$5" library="SRD-05VDC-SL-C" deviceset="RELAY" device="PTH"/>
-<part name="D1" library="diode" library_urn="urn:adsk.eagle:library:210" deviceset="1N4004" device="" package3d_urn="urn:adsk.eagle:package:43336/1"/>
+<part name="RL1" library="SRD-05VDC-SL-C" deviceset="RELAY" device="PTH"/>
+<part name="D1" library="diode" library_urn="urn:adsk.eagle:library:210" deviceset="1N4004" device="" package3d_urn="urn:adsk.eagle:package:43336/1" value="1N4007"/>
 <part name="R2" library="resistor" library_urn="urn:adsk.eagle:library:348" deviceset="R-EU_" device="0309/10" package3d_urn="urn:adsk.eagle:package:23567/1" value="1K"/>
 <part name="R3" library="resistor" library_urn="urn:adsk.eagle:library:348" deviceset="R-EU_" device="0309/10" package3d_urn="urn:adsk.eagle:package:23567/1" value="1K"/>
@@
 <attribute name="VALUE" x="39.37" y="54.102" size="1.778" layer="96" rot="R180"/>
 </instance>
-<instance part="LED5" gate="G$1" x="15.24" y="50.8" smashed="yes" rot="R90">
+<instance part="LED2" gate="G$1" x="15.24" y="50.8" smashed="yes" rot="R90">
 <attribute name="NAME" x="19.812" y="54.356" size="1.778" layer="95" rot="R180"/>
 <attribute name="VALUE" x="19.812" y="56.515" size="1.778" layer="96" rot="R180"/>
@@
 </instance>
 <instance part="U$4" gate="G$1" x="233.68" y="104.14" smashed="yes"/>
-<instance part="JP1" gate="1" x="2.54" y="7.62" smashed="yes" rot="R90">
+<instance part="RGB" gate="1" x="2.54" y="7.62" smashed="yes" rot="R90">
 <attribute name="NAME" x="2.54" y="3.81" size="1.778" layer="95" rot="R180"/>
 <attribute name="VALUE" x="2.54" y="13.335" size="1.778" layer="96" rot="R180"/>
@@
 <attribute name="VALUE" x="327.66" y="68.58" size="1.778" layer="96"/>
 </instance>
-<instance part="U$5" gate="G$1" x="340.36" y="48.26" smashed="yes">
+<instance part="RL1" gate="G$1" x="340.36" y="48.26" smashed="yes">
 <attribute name="NAME" x="332.74" y="56.388" size="1.778" layer="95"/>
 <attribute name="VALUE" x="332.74" y="38.1" size="1.778" layer="96"/>
@@
 <pinref part="CONFIG" gate="G$1" pin="1"/>
 <wire x1="5.08" y1="40.64" x2="12.7" y2="40.64" width="0.1524" layer="91"/>
-<pinref part="LED5" gate="G$1" pin="A"/>
+<pinref part="LED2" gate="G$1" pin="A"/>
 <wire x1="12.7" y1="50.8" x2="5.08" y2="50.8" width="0.1524" layer="91"/>
 <wire x1="5.08" y1="50.8" x2="5.08" y2="40.64" width="0.1524" layer="91"/>
@@
 <junction x="124.46" y="30.48"/>
 <junction x="114.3" y="63.5"/>
-<pinref part="JP1" gate="1" pin="3"/>
+<pinref part="RGB" gate="1" pin="3"/>
 <wire x1="5.08" y1="10.16" x2="5.08" y2="40.64" width="0.1524" layer="91"/>
 <junction x="5.08" y="40.64"/>
@@
 <wire x1="190.5" y1="73.66" x2="190.5" y2="99.06" width="0.1524" layer="91"/>
 <junction x="190.5" y="99.06"/>
-<pinref part="U$5" gate="G$1" pin="COIL0"/>
+<pinref part="RL1" gate="G$1" pin="COIL0"/>
 <wire x1="330.2" y1="43.18" x2="327.66" y2="43.18" width="0.1524" layer="91"/>
 <pinref part="D1" gate="1" pin="A"/>
@@
 <net name="N$18" class="0">
 <segment>
-<pinref part="LED5" gate="G$1" pin="C"/>
+<pinref part="LED2" gate="G$1" pin="C"/>
 <pinref part="R5" gate="G$1" pin="2"/>
 <wire x1="20.32" y1="50.8" x2="30.48" y2="50.8" width="0.1524" layer="91"/>
@@
 <wire x1="134.62" y1="124.46" x2="134.62" y2="86.36" width="0.1524" layer="91"/>
 <junction x="114.3" y="66.04"/>
-<pinref part="JP1" gate="1" pin="2"/>
+<pinref part="RGB" gate="1" pin="2"/>
 <wire x1="134.62" y1="86.36" x2="134.62" y2="66.04" width="0.1524" layer="91"/>
 <wire x1="5.08" y1="7.62" x2="48.26" y2="7.62" width="0.1524" layer="91"/>
@@
 <net name="N$1" class="0">
 <segment>
-<pinref part="JP1" gate="1" pin="1"/>
+<pinref part="RGB" gate="1" pin="1"/>
 <wire x1="5.08" y1="5.08" x2="53.34" y2="5.08" width="0.1524" layer="91"/>
 <pinref part="U$2" gate="G$1" pin="D7"/>
@@
 <net name="N$12" class="0">
 <segment>
-<pinref part="U$5" gate="G$1" pin="COIL1"/>
+<pinref part="RL1" gate="G$1" pin="COIL1"/>
 <wire x1="327.66" y1="53.34" x2="330.2" y2="53.34" width="0.1524" layer="91"/>
 <pinref part="D1" gate="1" pin="C"/>
@@
 <wire x1="213.36" y1="96.52" x2="213.36" y2="33.02" width="0.1524" layer="91"/>
 <wire x1="213.36" y1="33.02" x2="358.14" y2="33.02" width="0.1524" layer="91"/>
-<pinref part="U$5" gate="G$1" pin="SWCOMMON"/>
+<pinref part="RL1" gate="G$1" pin="SWCOMMON"/>
 <wire x1="358.14" y1="33.02" x2="358.14" y2="48.26" width="0.1524" layer="91"/>
 <wire x1="358.14" y1="48.26" x2="347.98" y2="48.26" width="0.1524" layer="91"/>
@@
 <wire x1="215.9" y1="25.4" x2="215.9" y2="5.08" width="0.1524" layer="91"/>
 <pinref part="X3" gate="-2" pin="1"/>
-<pinref part="U$5" gate="G$1" pin="SWCLOSE"/>
+<pinref part="RL1" gate="G$1" pin="SWCLOSE"/>
 <wire x1="360.68" y1="25.4" x2="360.68" y2="53.34" width="0.1524" layer="91"/>
 <wire x1="360.68" y1="53.34" x2="347.98" y2="53.34" width="0.1524" layer="91"/>
@@
 <wire x1="220.98" y1="20.32" x2="220.98" y2="5.08" width="0.1524" layer="91"/>
 <wire x1="355.6" y1="20.32" x2="355.6" y2="43.18" width="0.1524" layer="91"/>
-<pinref part="U$5" gate="G$1" pin="SWOPEN"/>
+<pinref part="RL1" gate="G$1" pin="SWOPEN"/>
 <wire x1="355.6" y1="43.18" x2="347.98" y2="43.18" width="0.1524" layer="91"/>
 </segment>
