File: HB-OU-MP3-LED/EAGLE/HB-OU-MP3-LED_V1.3.brd (EAGLE design)
At the start: 76.2 x 100 mm, 22 parts, among them Q1 BC327, X1 MSTBA2, X3 MSTBA3

Commit message: Update HB-OU-MP3-LED_V1.3.brd
Parts:
- added R1: 10K, resistor:0309/10
Connections:
- new net N$21: LED1.K, OK1.1
- new net N$22: Q1.2, R4.2
- net GND: now also R1.1; no longer LED1.K, OK1.3
- net N$13: now also U$5.SWCLOSED; no longer U$5.SWCOMMON
- net N$16: now also OK1.3, R1.2, R4.1; no longer OK1.4, Q1.2, R4.2
- net N$7: now also U$5.SWCOMMON; no longer U$5.SWCLOSED
- net N$8: no longer OK1.1
- net RAW: now also OK1.4; no longer R4.1
Routing:
- net N$8: track 34.7 -> 0.00 mm
- net GND: track 265.5 -> 246.0 mm
- net RAW: track 103.1 -> 87.9 mm
- net N$16: track 9.79 -> 0.00 mm
- net N$13: track 15.8 -> 10.6 mm
- net N$20: track 34.0 -> 30.9 mm
- net N$7: track 18.2 -> 16.5 mm
Changed lines of the file:
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@@
 <attribute name="POPULARITY" value="3" x="2.54" y="16.51" size="1.778" layer="27" rot="R270" display="off"/>
+</element>
+<element name="R1" library="resistor" library_urn="urn:adsk.eagle:library:348" package="0309/10" package3d_urn="urn:adsk.eagle:package:23567/1" value="10K" x="3.81" y="-3.81" smashed="yes">
+<attribute name="NAME" x="-0.381" y="-1.905" size="1.27" layer="25" ratio="10"/>
+<attribute name="VALUE" x="0.635" y="-4.4958" size="1.27" layer="27" ratio="10"/>
 </element>
 </elements>
@@
 <contactref element="D1" pad="A"/>
 <contactref element="OK1" pad="2"/>
-<contactref element="OK1" pad="3"/>
-<contactref element="LED1" pad="K"/>
-<wire x1="19.05" y1="34.29" x2="26.67" y2="34.29" width="0.254" layer="16"/>
-<wire x1="19.05" y1="34.29" x2="11.43" y2="34.29" width="0.254" layer="16"/>
 <wire x1="11.43" y1="34.29" x2="6.35" y2="34.29" width="0.254" layer="16"/>
 <wire x1="6.35" y1="34.29" x2="5.08" y2="35.56" width="0.254" layer="16"/>
@@
 <wire x1="71.12" y1="7.62" x2="67.31" y2="7.62" width="0.254" layer="16"/>
 <wire x1="66.04" y1="31.75" x2="72.39" y2="25.4" width="0.254" layer="16"/>
-<wire x1="43.18" y1="5.08" x2="45.72" y2="5.08" width="0.254" layer="16"/>
 <wire x1="48.26" y1="7.62" x2="49.53" y2="7.62" width="0.254" layer="16"/>
 <wire x1="45.72" y1="5.08" x2="48.26" y2="7.62" width="0.254" layer="16"/>
-<wire x1="43.18" y1="5.08" x2="41.91" y2="3.81" width="0.254" layer="16"/>
 <wire x1="26.59" y1="3.81" x2="23.82" y2="6.58" width="0.254" layer="16"/>
 <wire x1="41.91" y1="3.81" x2="26.59" y2="3.81" width="0.254" layer="16"/>
@@
 <wire x1="52.07" y1="64.77" x2="50.8" y2="63.5" width="0.254" layer="1"/>
 <wire x1="50.8" y1="63.5" x2="45.72" y2="63.5" width="0.254" layer="1"/>
+<contactref element="R1" pad="1"/>
+<wire x1="11.43" y1="34.29" x2="26.67" y2="34.29" width="0" layer="19" extent="16-16"/>
+<wire x1="45.72" y1="5.08" x2="41.91" y2="3.81" width="0" layer="19" extent="16-16"/>
+<wire x1="-1.27" y1="-3.81" x2="5.08" y2="7.62" width="0" layer="19" extent="16-16"/>
 </signal>
 <signal name="N$17">
@@
 <contactref element="JP1" pad="2"/>
 <contactref element="Q1" pad="1"/>
-<contactref element="R4" pad="1"/>
 <wire x1="63.5" y1="75.1078" x2="63.5" y2="71.12" width="0.254" layer="16"/>
 <wire x1="63.5" y1="71.12" x2="58.42" y2="66.04" width="0.254" layer="16"/>
 <wire x1="58.42" y1="66.04" x2="45.72" y2="66.04" width="0.254" layer="16"/>
-<wire x1="5.08" y1="38.1" x2="13.97" y2="38.1" width="0.254" layer="1"/>
-<wire x1="13.97" y1="38.1" x2="20.32" y2="38.1" width="0.254" layer="1"/>
 <wire x1="20.32" y1="38.1" x2="21.59" y2="36.83" width="0.254" layer="1"/>
 <wire x1="21.59" y1="36.83" x2="21.59" y2="26.67" width="0.254" layer="1"/>
@@
 <wire x1="33.02" y1="35.56" x2="29.21" y2="35.56" width="0.254" layer="1"/>
 <wire x1="29.21" y1="35.56" x2="26.67" y2="38.1" width="0.254" layer="1"/>
+<contactref element="OK1" pad="4"/>
+<wire x1="21.59" y1="36.83" x2="19.05" y2="31.75" width="0" layer="19" extent="1-1"/>
+<wire x1="5.08" y1="38.1" x2="20.32" y2="38.1" width="0" layer="19" extent="1-1"/>
 </signal>
 <signal name="N$10">
@@
 <signal name="N$7">
 <contactref element="U$4" pad="SPK2"/>
-<contactref element="U$5" pad="SWCLOSED"/>
 <wire x1="49.53" y1="5.08" x2="49.53" y2="3.81" width="0.254" layer="1"/>
 <wire x1="49.53" y1="3.81" x2="48.26" y2="2.54" width="0.254" layer="1"/>
 <wire x1="48.26" y1="2.54" x2="38.1" y2="2.54" width="0.254" layer="1"/>
-<wire x1="35.82" y1="4.82" x2="35.82" y2="6.58" width="0.254" layer="1"/>
 <wire x1="38.1" y1="2.54" x2="35.82" y2="4.82" width="0.254" layer="1"/>
+<contactref element="U$5" pad="SWCOMMON"/>
+<wire x1="21.82" y1="12.58" x2="35.82" y2="4.82" width="0" layer="19" extent="1-1"/>
 </signal>
 <signal name="N$13">
-<contactref element="U$5" pad="SWCOMMON"/>
 <contactref element="X3" pad="2"/>
-<wire x1="21.82" y1="12.58" x2="16.63" y2="12.58" width="0.254" layer="16"/>
 <wire x1="16.63" y1="12.58" x2="12.7" y2="16.51" width="0.254" layer="16"/>
 <wire x1="12.7" y1="16.51" x2="7.62" y2="16.51" width="0.254" layer="16"/>
+<contactref element="U$5" pad="SWCLOSED"/>
+<wire x1="16.63" y1="12.58" x2="35.82" y2="6.58" width="0" layer="19" extent="16-16"/>
 </signal>
 <signal name="N$14">
@@
 <wire x1="48.26" y1="17.78" x2="49.53" y2="17.78" width="0.254" layer="16"/>
 </signal>
-<signal name="N$16">
-<contactref element="R4" pad="2"/>
-<contactref element="OK1" pad="4"/>
-<contactref element="Q1" pad="2"/>
-<wire x1="13.97" y1="27.94" x2="18.415" y2="27.94" width="0.254" layer="16"/>
-<wire x1="18.415" y1="27.94" x2="19.05" y2="27.305" width="0.254" layer="16"/>
-<wire x1="19.05" y1="31.75" x2="19.05" y2="27.305" width="0.254" layer="16"/>
+<signal name="N$20">
+<contactref element="X3" pad="3"/>
+<wire x1="35.82" y1="15.5" x2="30.48" y2="10.16" width="0.254" layer="16"/>
+<wire x1="30.48" y1="10.16" x2="8.89" y2="10.16" width="0.254" layer="16"/>
+<wire x1="8.89" y1="10.16" x2="7.62" y2="11.43" width="0.254" layer="16"/>
+<contactref element="U$5" pad="SWOPEN"/>
+<wire x1="35.82" y1="15.5" x2="35.82" y2="18.58" width="0" layer="19" extent="16-16"/>
 </signal>
 <signal name="N$8">
 <contactref element="R6" pad="2"/>
 <contactref element="LED1" pad="A"/>
+<wire x1="43.18" y1="7.62" x2="43.18" y2="10.16" width="0" layer="19" extent="1-1"/>
+</signal>
+<signal name="N$21">
+<contactref element="LED1" pad="K"/>
 <contactref element="OK1" pad="1"/>
-<wire x1="43.18" y1="10.16" x2="43.18" y2="7.62" width="0.254" layer="16"/>
-<wire x1="26.67" y1="31.75" x2="26.67" y2="25.4" width="0.254" layer="16"/>
-<wire x1="43.18" y1="15.24" x2="43.18" y2="10.16" width="0.254" layer="16"/>
-<wire x1="26.67" y1="25.4" x2="30.48" y2="21.59" width="0.254" layer="16"/>
-<wire x1="30.48" y1="21.59" x2="36.83" y2="21.59" width="0.254" layer="16"/>
-<wire x1="36.83" y1="21.59" x2="43.18" y2="15.24" width="0.254" layer="16"/>
-</signal>
-<signal name="N$20">
-<contactref element="U$5" pad="SWOPEN"/>
-<contactref element="X3" pad="3"/>
-<wire x1="35.82" y1="18.58" x2="35.82" y2="15.5" width="0.254" layer="16"/>
-<wire x1="35.82" y1="15.5" x2="30.48" y2="10.16" width="0.254" layer="16"/>
-<wire x1="30.48" y1="10.16" x2="8.89" y2="10.16" width="0.254" layer="16"/>
-<wire x1="8.89" y1="10.16" x2="7.62" y2="11.43" width="0.254" layer="16"/>
+<wire x1="43.18" y1="5.08" x2="26.67" y2="31.75" width="0" layer="19" extent="1-1"/>
+</signal>
+<signal name="N$16">
+<contactref element="OK1" pad="3"/>
+<contactref element="R4" pad="1"/>
+<contactref element="R1" pad="2"/>
+<wire x1="13.97" y1="38.1" x2="19.05" y2="34.29" width="0" layer="19" extent="1-1"/>
+<wire x1="8.89" y1="-3.81" x2="19.05" y2="34.29" width="0" layer="19" extent="1-1"/>
+</signal>
+<signal name="N$22">
+<contactref element="R4" pad="2"/>
+<contactref element="Q1" pad="2"/>
+<wire x1="13.97" y1="27.94" x2="19.05" y2="27.305" width="0" layer="19" extent="1-1"/>
 </signal>
 </signals>

Commit message: Update HB-OU-MP3-LED_V1.3.brd
Parts:
- moved R1 48.2 mm to (19.1, 41.9), turned to 270 degrees
Routing:
- net N$21: track 0.00 -> 37.2 mm
- net N$13: track 10.6 -> 33.8 mm, vias 0 -> 1
- net GND: track 246.0 -> 266.3 mm
- net N$7: track 16.5 -> 36.6 mm
- net RAW: track 87.9 -> 101.9 mm
- net N$16: track 0.00 -> 8.15 mm
- net N$22: track 0.00 -> 5.34 mm
- net N$20: track 30.9 -> 34.0 mm
- net N$8: track 0.00 -> 2.54 mm

Commit message: Update HB-OU-MP3-LED_V1.3.brd
Parts:
- D1: value 1N4004 -> 1N4007
- renumbered JP1 to RGB, LED5 to LED2, U$5 to RL1
Other:
- board text added: "CC1101"
